File: test/cli/bundle/reference/pcbs/pcb.kicad_pcb (KiCad board)
At the start: 2 copper layers, 18 x 18 mm, 1 part

Commit message: TEST: Fix tests for new power netclass
Other:
- net class Power added: clearance 0.2, trace_width 0.5, via_dia 0.8, via_drill 0.4
Changed lines of the file:
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@@
     (add_net "")
+  )
+  (net_class Power "This is the power net class."
+    (clearance 0.2)
+    (trace_width 0.5)
+    (via_dia 0.8)
+    (via_drill 0.4)
+    (uvia_dia 0.3)
+    (uvia_drill 0.1)
   )
     (module injected_test_footprint (layer F.Cu)
