File: test/footprints/rest___pcbs_pcb.kicad_pcb (KiCad board)
At the start: 2 copper layers, 2.4 x 14.2 mm, 10 parts, among them J1 Jumper

Commit message: TEST: Fix tests for new power netclass
Parts:
- removed the REF** at (0.00, -150.0)
- added _1: VIA-0.6mm, VIA-0.6mm, F.Cu at (0.00, -150.0)
- J1: footprint lib:Jumper -> PCM12SMTR
Other:
- net class Power added: clearance 0.2, trace_width 0.5, via_dia 0.8, via_drill 0.4
Changed lines of the file:
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@@
 (add_net "pos")
 (add_net "neg")
-(add_net "VCC")
-(add_net "GND")
 (add_net "SDA")
 (add_net "SCL")
@@
 (add_net "D")
 (add_net "net")
+  )
+  (net_class Power "This is the power net class."
+    (clearance 0.2)
+    (trace_width 0.5)
+    (via_dia 0.8)
+    (via_drill 0.4)
+    (uvia_dia 0.3)
+    (uvia_drill 0.1)
+    (add_net "VCC")
+(add_net "GND")
   )
     (module ALPS (layer F.Cu)
@@
         (pad 2 thru_hole oval (at 1 0 0) (size 1.2 1.7) (drill 0.75) (layers *.Cu *.Mask) (net 4 "neg"))
     )
-        (module lib:Jumper (layer F.Cu)
+        (footprint "PCM12SMTR" (layer F.Cu)
         (at 100 0 0)
         (fp_text reference "J1" (at 0 0) (layer F.SilkS) hide (effects (font (size 1.27 1.27) (thickness 0.15))))
         (fp_text value Jumper (at 0 -7.3) (layer F.Fab) (effects (font (size 1 1) (thickness 0.15))))
+        (fp_text value Jumper (at 0 2 270) (layer F.SilkS) (effects (font (size 1 1) (thickness 0.15))  ))
         (pad 1 smd rect (at -0.50038 0 0) (size 0.635 1.143) (layers F.Cu F.Paste F.Mask)
         (clearance 0.1905) (net 1 "from"))
@@
             (pad "" thru_hole rect (at -0.12 5.56 0)  (size 3.2 2) (drill oval 2.8 1.5) (layers *.Cu *.Mask))
         )
-        (module RollerEncoder_Panasonic_EVQWGD001 (layer F.Cu)
+        (module RollerEncoder_Panasonic_EVQWGD001 (layer "F.Cu")
         (at 50 -100 0)
-        (fp_text reference REF** (at 0 0 0) (layer F.Fab) (effects (font (size 1 1) (thickness 0.15))))
-        (fp_text value RollerEncoder_Panasonic_EVQWGD001 (at -0.1 9 0) (layer F.Fab) (effects (font (size 1 1) (thickness 0.15))))
-        (fp_line (start -8.4 -6.4) (end 8.4 -6.4) (layer Dwgs.User) (width 0.12))
-        (fp_line (start 8.4 -6.4) (end 8.4 7.4) (layer Dwgs.User) (width 0.12))
-        (fp_line (start 8.4 7.4) (end -8.4 7.4) (layer Dwgs.User) (width 0.12))
-        (fp_line (start -8.4 7.4) (end -8.4 -6.4) (layer Dwgs.User) (width 0.12))
-          (fp_line (start 9.8 7.3) (end 9.8 -6.3) (layer Edge.Cuts) (width 0.15))
-          (fp_line (start 7.4 -6.3) (end 7.4 7.3) (layer Edge.Cuts) (width 0.15))
-          (fp_line (start 9.5 -6.6) (end 7.7 -6.6) (layer Edge.Cuts) (width 0.15))
-          (fp_line (start 7.7 7.6) (end 9.5 7.6) (layer Edge.Cuts) (width 0.15))
-          (fp_arc (start 7.7 7.3) (end 7.4 7.3) (angle -90) (layer Edge.Cuts) (width 0.15))
-          (fp_arc (start 9.5 7.3) (end 9.5 7.6) (angle -90) (layer Edge.Cuts) (width 0.15))
-          (fp_arc (start 7.7 -6.3) (end 7.7 -6.6) (angle -90) (layer Edge.Cuts) (width 0.15))
-          (fp_arc (start 9.5 -6.3) (end 9.8 -6.3) (angle -90) (layer Edge.Cuts) (width 0.15))
-          (pad S1 thru_hole circle (at -6.85 -6.2 0) (size 1.6 1.6) (drill 0.9) (layers *.Cu *.Mask) (net 1 "from"))
-          (pad S2 thru_hole circle (at -5 -6.2 0) (size 1.6 1.6) (drill 0.9) (layers *.Cu *.Mask) (net 2 "to"))
-          (pad A thru_hole circle (at -5.625 -3.81 0) (size 1.6 1.6) (drill 0.9) (layers *.Cu *.Mask) (net 11 "A"))
-          (pad B thru_hole circle (at -5.625 -1.27 0) (size 1.6 1.6) (drill 0.9) (layers *.Cu *.Mask) (net 12 "B"))
-          (pad C thru_hole circle (at -5.625 1.27 0) (size 1.6 1.6) (drill 0.9) (layers *.Cu *.Mask) (net 13 "C"))
-          (pad D thru_hole circle (at -5.625 3.81 0) (size 1.6 1.6) (drill 0.9) (layers *.Cu *.Mask) (net 14 "D"))
+        (attr through_hole)
+        (fp_text reference REF** (at 0 0 0) (layer "F.Fab") (effects (font (size 1 1) (thickness 0.15))))
+        (fp_text value RollerEncoder_Panasonic_EVQWGD001 (at -0.1 9 0) (layer "F.Fab") (effects (font (size 1 1) (thickness 0.15))))
+        (fp_line (start -8.4 -6.4) (end 8.4 -6.4) (layer "Dwgs.User") (width 0.12))
+        (fp_line (start 8.4 -6.4) (end 8.4 7.4) (layer "Dwgs.User") (width 0.12))
+        (fp_line (start 8.4 7.4) (end -8.4 7.4) (layer "Dwgs.User") (width 0.12))
+        (fp_line (start -8.4 7.4) (end -8.4 -6.4) (layer "Dwgs.User") (width 0.12))
+         (fp_line (start 9.8 7.3) (end 9.8 -6.3) (layer "Edge.Cuts") (width 0.15))
+         (fp_line (start 7.4 -6.3) (end 7.4 7.3) (layer "Edge.Cuts") (width 0.15))
+         (fp_line (start 9.5 -6.6) (end 7.7 -6.6) (layer "Edge.Cuts") (width 0.15))
+         (fp_line (start 7.7 7.6) (end 9.5 7.6) (layer "Edge.Cuts") (width 0.15))
+         (fp_arc (start 9.8 7.3) (mid 9.712132 7.512132) (end 9.5 7.6) (layer "Edge.Cuts") (width 0.15))
+         (fp_arc (start 7.7 7.6) (mid 7.487868 7.512132) (end 7.4 7.3) (layer "Edge.Cuts") (width 0.15))
+         (fp_arc (start 9.5 -6.6) (mid 9.712132 -6.512132) (end 9.8 -6.3) (layer "Edge.Cuts") (width 0.15))
+         (fp_arc (start 7.4 -6.3) (mid 7.487868 -6.512132) (end 7.7 -6.6) (layer "Edge.Cuts") (width 0.15))
+          (pad "S1" thru_hole circle (at -6.85 -6.2 0) (size 1.6 1.6) (drill 0.9) (layers *.Cu *.Mask) (net 1 "from"))
+          (pad "S2" thru_hole circle (at -5 -6.2 0) (size 1.6 1.6) (drill 0.9) (layers *.Cu *.Mask) (net 2 "to"))
+          (pad "A" thru_hole circle (at -5.625 -3.81 0) (size 1.6 1.6) (drill 0.9) (layers *.Cu *.Mask) (net 11 "A"))
+          (pad "B" thru_hole circle (at -5.625 -1.27 0) (size 1.6 1.6) (drill 0.9) (layers *.Cu *.Mask) (net 12 "B"))
+          (pad "C" thru_hole circle (at -5.625 1.27 0) (size 1.6 1.6) (drill 0.9) (layers *.Cu *.Mask) (net 13 "C"))
+          (pad "D" thru_hole circle (at -5.625 3.81 0) (size 1.6 1.6) (drill 0.9) (layers *.Cu *.Mask) (net 14 "D"))
           (pad "" np_thru_hole circle (at -5.625 6.3 0) (size 1.5 1.5) (drill 1.5) (layers *.Cu *.Mask))
         )
@@
       (module VIA-0.6mm (layer F.Cu)
       (at 0 -150 0)
-      (fp_text reference REF** (at 0 1.4) (layer F.SilkS) hide (effects (font (size 1 1) (thickness 0.15))))
+      (fp_text reference _1 (at 0 1.4) (layer F.SilkS) hide (effects (font (size 1 1) (thickness 0.15))))
       (fp_text value VIA-0.6mm (at 0 -1.4) (layer F.Fab) hide (effects (font (size 1 1) (thickness 0.15))))
       (pad 1 thru_hole circle (at 0 0) (size 0.6 0.6) (drill 0.3) (layers *.Cu) (zone_connect 2) (net 15 "net"))
