File: test/pcbs/mock_footprints___pcbs_main.kicad_pcb (KiCad board)
At the start: 2 copper layers, 39 x 19 mm, 7 parts

Commit message: TEST: Fix tests for new power netclass
Parts:
- removed the ? at (1.00, -1.00) (x2)
- removed the ? at (19.0, -1.00) (x2)
- added ? (x2): , trace_test, F.Cu at (1.00, -1.00)
- added ? (x2): , trace_test, B.Cu at (19.0, -1.00)
Other:
- net class Power added: clearance 0.2, trace_width 0.5, via_dia 0.8, via_drill 0.4
Changed lines of the file:
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@@
 (add_net "T6_3")
+  )
+  (net_class Power "This is the power net class."
+    (clearance 0.2)
+    (trace_width 0.5)
+    (via_dia 0.8)
+    (via_drill 0.4)
+    (uvia_dia 0.3)
+    (uvia_drill 0.1)
   )
                 (module trace_test (layer F.Cu)
